File: hard/pcb_main/e4.sch (EAGLE design)
At the start: 1 part

Commit message: nop
Parts:
- added U$2: (no value), connector:GENERIC_10_XP
- added XP2: (no value), connector:GENERIC_04_XP
- added XP3: (no value), connector:GENERIC_32_XP
- added XS1: (no value), connector:GENERIC_32_XS
- added XS10, XS11, XS3: (no value), connector:GENERIC_08_XS
- added XS12: (no value), connector:GENERIC_10_XS
- added XS2: (no value), connector:GENERIC_19_XS
- added XS4, XS5, XS6, XS7, XS8: (no value), connector:GENERIC_16_XS
- added XS9: (no value), connector:GENERIC_34_XS
- XP1: value (none) -> 2PM_19pin; device connector:GENERIC_32 -> connector:GENERIC_19_XP
Connections:
- new net +24: XP2.1, XP2.2, XS3.2, XS3.4, XS3.6, XS3.8
- new net AN10: XS8.10
- new net AN11: XS8.11
- new net AN12: XS8.12
- new net AN13: XS8.13
- new net AN14: XS8.14
- new net AN15: XS8.15
- new net AN16: XS8.16
- new net AN2: XS8.2
- new net AN3: XS8.3
- new net AN4: XS8.4
- new net AN5: XS8.5
- new net AN6: XS8.6
- new net AN7: XS8.7
- new net AN8: XS8.8
- new net AN9: XS8.9
- new net GND: XP2.3, XP2.4, XS3.1, XS3.3, XS3.5, XS3.7
- new net OUT_DRV1: XS2.1, XS9.1, XS9.4
- new net OUT_DRV2: XS2.3, XS9.5, XS9.8
- new net OUT_DRV3: XS2.5, XS9.12, XS9.9
- new net OUT_DRV4: XS2.7, XS9.13, XS9.16
- new net OUT_DRV5: XS2.9, XS9.17, XS9.20
- new net OUT_DRV6: XS2.11, XS9.21, XS9.24
- new net OUT_DRV7: XS2.13, XS9.25, XS9.28
- new net OUT_DRV8: XS2.15, XS9.29, XS9.32
- new net REL1: XS1.1, XS4.1
- new net REL10: XS1.10, XS4.10
- new net REL11: XS1.11, XS4.11
- new net REL12: XS1.12, XS4.12
- new net REL13: XS1.13, XS4.13
- new net REL14: XS1.14, XS4.14
- new net REL15: XS1.15, XS4.15
- new net REL16: XS1.16, XS4.16
- new net REL17: XS1.17, XS5.1
- new net REL18: XS1.18, XS5.2
- new net REL19: XS1.19, XS5.3
- new net REL2: XS1.2, XS4.2
- new net REL20: XS1.20, XS5.4
- new net REL21: XS1.21, XS5.5
- new net REL22: XS1.22, XS5.6
- new net REL23: XS1.23, XS5.7
- new net REL24: XS1.24, XS5.8
- new net REL25: XS1.25, XS5.9
- new net REL26: XS1.26, XS5.10
- new net REL27: XS1.27, XS5.11
- new net REL28: XS1.28, XS5.12
- new net REL29: XS1.29, XS5.13
- new net REL3: XS1.3, XS4.3
- new net REL30: XS1.30, XS5.14
- new net REL31: XS1.31, XS5.15
- new net REL32: XS1.32, XS5.16
- new net REL33: XP3.1, XS6.1
- new net REL34: XP3.2, XS6.2
- new net REL35: XP3.3, XS6.3
- new net REL36: XP3.4, XS6.4
- new net REL37: XP3.5, XS6.5
- new net REL38: XP3.6, XS6.6
- new net REL39: XP3.7, XS6.7
- new net REL4: XS1.4, XS4.4
- new net REL40: XP3.8, XS6.8
- new net REL41: XP3.9, XS6.9
- new net REL42: XP3.10, XS6.10
- new net REL43: XP3.11, XS6.11
- new net REL44: XP3.12, XS6.12
- new net REL45: XP3.13, XS6.13
- new net REL46: XP3.14, XS6.14
- new net REL47: XP3.15, XS6.15
- new net REL48: XP3.16, XS6.16
- new net REL49: XP3.17, XS7.1
- new net REL5: XS1.5, XS4.5
- new net REL50: XP3.18, XS7.2
- new net REL51: XP3.19, XS7.3
- new net REL52: XP3.20, XS7.4
- new net REL53: XP3.21, XS7.5
- new net REL54: XP3.22, XS7.6
- new net REL55: XP3.23, XS7.7
- new net REL56: XP3.24, XS7.8
- new net REL57: XP3.25, XS7.9
- new net REL58: XP3.26, XS7.10
- new net REL59: XP3.27, XS7.11
- new net REL6: XS1.6, XS4.6
- new net REL60: XP3.28, XS7.12
- new net REL61: XP3.29, XS7.13
- new net REL62: XP3.30, XS7.14
- new net REL63: XP3.31, XS7.15
- new net REL64: XP3.32, XS7.16
- new net REL7: XS1.7, XS4.7
- new net REL8: XS1.8, XS4.8
- new net REL9: XS1.9, XS4.9
- new net VCC_DRV1: XS2.2, XS9.2, XS9.3
- new net VCC_DRV2: XS2.4, XS9.6, XS9.7
- new net VCC_DRV3: XS2.6, XS9.10, XS9.11
- new net VCC_DRV4: XS2.8, XS9.14, XS9.15
- new net VCC_DRV5: XS2.10, XS9.18, XS9.19
- new net VCC_DRV6: XS2.12, XS9.22, XS9.23
- new net VCC_DRV7: XS2.14, XS9.26, XS9.27
- new net VCC_DRV8: XS2.16, XS9.30, XS9.31
- net AN1: now also XS8.1; no longer XP1.1
Other:
- note added: "AN1"
- note added: "AN10"
- note added: "AN11"
- note added: "AN12"
- note added: "AN13"
- note added: "AN14"
- note added: "AN15"
- note added: "AN16"
- note added: "AN2"
- note added: "AN3"
- note added: "AN4"
- note added: "AN5"
- note added: "AN6"
- note added: "AN7"
- note added: "AN8"
- note added: "AN9"
- note removed: "REL01"
