File: hard/pcb_main/main.brd (EAGLE design)
At the start: 210 x 132 mm, 817 parts

Commit message: fixed name
Parts:
- moved C1 0.35 mm to (41.8, 71.2)
Routing:
- net JTMS: track 39.9 -> 38.6 mm
- net GND: vias 115 -> 120
Changed lines of the file:
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@@
 <setting verticaltext="up"/>
 </settings>
-<grid distance="0.5" unitdist="mm" unit="mm" style="lines" multiple="1" display="yes" altdistance="0.005" altunitdist="inch" altunit="inch"/>
+<grid distance="0.25" unitdist="mm" unit="mm" style="lines" multiple="1" display="yes" altdistance="0.005" altunitdist="inch" altunit="inch"/>
 <layers>
 <layer number="1" name="Top" color="4" fill="1" visible="yes" active="yes"/>
@@
 <layer number="23" name="tOrigins" color="15" fill="1" visible="yes" active="yes"/>
 <layer number="24" name="bOrigins" color="15" fill="1" visible="yes" active="yes"/>
-<layer number="25" name="tNames" color="7" fill="1" visible="yes" active="yes"/>
-<layer number="26" name="bNames" color="15" fill="1" visible="yes" active="yes"/>
+<layer number="25" name="tNames" color="7" fill="1" visible="no" active="yes"/>
+<layer number="26" name="bNames" color="15" fill="1" visible="no" active="yes"/>
 <layer number="27" name="tValues" color="7" fill="1" visible="no" active="yes"/>
 <layer number="28" name="bValues" color="7" fill="1" visible="no" active="yes"/>
-<layer number="29" name="tStop" color="7" fill="3" visible="yes" active="yes"/>
-<layer number="30" name="bStop" color="7" fill="6" visible="yes" active="yes"/>
+<layer number="29" name="tStop" color="7" fill="3" visible="no" active="yes"/>
+<layer number="30" name="bStop" color="7" fill="6" visible="no" active="yes"/>
 <layer number="31" name="tCream" color="7" fill="4" visible="no" active="yes"/>
 <layer number="32" name="bCream" color="7" fill="5" visible="no" active="yes"/>
@@
 </element>
 <element name="DA12" library="vreg" package="TO263-5" value="LM2596S-5.0" x="182.15" y="49.05" smashed="yes" rot="R180">
-<attribute name="PARTNO" value="LM2596S-5.0" x="161.83" y="99.85" size="1.778" layer="27" rot="R180" display="off"/>
+<attribute name="PARTNO" value="LM2596S-5.0/NOPB" x="161.83" y="99.85" size="1.778" layer="27" rot="R180" display="off"/>
 <attribute name="NAME" x="175.1825" y="49.0075" size="1.016" layer="25" ratio="18" rot="R270"/>
 <attribute name="VALUE" x="175.165" y="53.5075" size="0.8128" layer="27" ratio="10" rot="R270"/>
 </element>
 <element name="DA13" library="vreg" package="TO263-5" value="LM2596S-5.0" x="177.769" y="31.153" smashed="yes" rot="R90">
-<attribute name="PARTNO" value="LM2596S-5.0" x="228.569" y="66.713" size="1.778" layer="27" rot="R90" display="off"/>
+<attribute name="PARTNO" value="LM2596S-5.0/NOPB" x="228.569" y="66.713" size="1.778" layer="27" rot="R90" display="off"/>
 <attribute name="NAME" x="178.3515" y="37.9955" size="1.016" layer="25" ratio="18" rot="R180"/>
 <attribute name="VALUE" x="182.2265" y="38.138" size="0.8128" layer="27" ratio="10" rot="R180"/>
@@
 <attribute name="VALUE" x="30.02055625" y="76.92450625" size="0.8128" layer="27" ratio="10" rot="R135"/>
 </element>
-<element name="C1" library="rcl" package="C0603" value="0.1uF" x="41.5" y="71.5" smashed="yes" rot="R45">
-<attribute name="DATABASE" value="./bom/volat3-PARTSDB.tsv" x="41.5" y="71.5" size="1.778" layer="27" rot="R45" display="off"/>
-<attribute name="PARTNO" value="C0603C104K5RACTU" x="41.5" y="71.5" size="1.778" layer="27" rot="R45" display="off"/>
-<attribute name="NAME" x="40.040671875" y="71.163275" size="1.016" layer="25" ratio="18" rot="R45"/>
-<attribute name="VALUE" x="41.72450625" y="69.479440625" size="0.8128" layer="27" ratio="10" rot="R45"/>
+<element name="C1" library="rcl" package="C0603" value="0.1uF" x="41.75" y="71.25" smashed="yes" rot="R45">
+<attribute name="DATABASE" value="./bom/volat3-PARTSDB.tsv" x="41.75" y="71.25" size="1.778" layer="27" rot="R45" display="off"/>
+<attribute name="PARTNO" value="C0603C104K5RACTU" x="41.75" y="71.25" size="1.778" layer="27" rot="R45" display="off"/>
+<attribute name="NAME" x="40.290671875" y="70.913275" size="1.016" layer="25" ratio="18" rot="R45"/>
+<attribute name="VALUE" x="41.97450625" y="69.229440625" size="0.8128" layer="27" ratio="10" rot="R45"/>
 </element>
 <element name="VD63" library="diode" package="SMB" value="SM6T200A" x="164.8" y="4.22" smashed="yes" rot="MR180">
@@
 <via x="57.023" y="49.276" extent="1-16" drill="0.5"/>
 <via x="55.023" y="54.776" extent="1-16" drill="0.5"/>
+<via x="42.75" y="73.25" extent="1-16" drill="0.5"/>
+<via x="18.5" y="63" extent="1-16" drill="0.5"/>
+<via x="36.5" y="81.25" extent="1-16" drill="0.5"/>
+<via x="41" y="75" extent="1-16" drill="0.5"/>
+<via x="63" y="79.25" extent="1-16" drill="0.5"/>
 </signal>
 <signal name="AN_RAW_0">
@@
 <wire x1="30.08461875" y1="74.045028125" x2="31" y2="73.129646875" width="0.3" layer="1"/>
 <wire x1="31" y1="73.129646875" x2="31" y2="72.5" width="0.3" layer="1"/>
-<wire x1="40.938696875" y1="70.938696875" x2="39.706209375" y2="70.938696875" width="0.3" layer="1"/>
-<wire x1="39.706209375" y1="70.938696875" x2="38.5699" y2="69.8023875" width="0.3" layer="1"/>
+<wire x1="41.188696875" y1="70.688696875" x2="39.456209375" y2="70.688696875" width="0.3" layer="1"/>
+<wire x1="39.456209375" y1="70.688696875" x2="38.5699" y2="69.8023875" width="0.3" layer="1"/>
 <wire x1="38.5699" y1="69.8023875" x2="38.5523875" y2="69.8023875" width="0.3" layer="1"/>
 <wire x1="40.337665625" y1="68.03461875" x2="40.337665625" y2="68.137665625" width="0.15" layer="1"/>
 <wire x1="40.337665625" y1="68.137665625" x2="41.2" y2="69" width="0.15" layer="1"/>
 <wire x1="41.2" y1="69" x2="41.2" y2="70.67739375" width="0.15" layer="1"/>
-<wire x1="41.2" y1="70.67739375" x2="40.938696875" y2="70.938696875" width="0.15" layer="1"/>
+<wire x1="41.2" y1="70.67739375" x2="41.188696875" y2="70.688696875" width="0.15" layer="1"/>
 <wire x1="21.0613" y1="65.0613" x2="21.350890625" y2="65.3113" width="0.3" layer="1"/>
 <wire x1="21.350890625" y1="65.3113" x2="22.30644375" y2="66.266853125" width="0.3" layer="1"/>
@@
 <wire x1="6.33" y1="36.25" x2="6.27" y2="36.19" width="0.15" layer="1"/>
 <wire x1="24.5" y1="54.25" x2="14.75" y2="44.5" width="0.15" layer="16"/>
-<wire x1="14.75" y1="44.5" x2="14.75" y2="36.25" width="0.15" layer="16"/>
-<wire x1="14.75" y1="36.25" x2="13.5" y2="35" width="0.15" layer="16"/>
-<wire x1="13.5" y1="35" x2="11.25" y2="35" width="0.15" layer="16"/>
+<wire x1="14.75" y1="44.5" x2="14.75" y2="38.75" width="0.15" layer="16"/>
 <via x="11.25" y="35" extent="1-16" drill="0.5"/>
 <wire x1="11.25" y1="35" x2="11.25" y2="36.0962" width="0.15" layer="1"/>
@@
 <wire x1="26.75" y1="52.5" x2="25" y2="54.25" width="0.15" layer="16"/>
 <wire x1="25" y1="54.25" x2="24.5" y2="54.25" width="0.15" layer="16"/>
+<wire x1="14.75" y1="38.75" x2="11.25" y2="35.25" width="0.15" layer="16"/>
+<wire x1="11.25" y1="35.25" x2="11.25" y2="35" width="0.15" layer="16"/>
 </signal>
 <signal name="JTCK">
@@
 <wire x1="37.463046875" y1="70.863046875" x2="36.3" y2="69.7" width="0.15" layer="1"/>
 <via x="36.3" y="69.7" extent="1-16" drill="0.5"/>
-<wire x1="30.75" y1="63" x2="15.75" y2="48" width="0.15" layer="16"/>
+<wire x1="30.75" y1="63" x2="14.1" y2="46.35" width="0.15" layer="16"/>
 <wire x1="36.3" y1="69.7" x2="34.45" y2="69.7" width="0.15" layer="16"/>
 <wire x1="34.45" y1="69.7" x2="33.5" y2="68.75" width="0.15" layer="16"/>
@@
 <via x="30.75" y="65.75" extent="1-16" drill="0.5"/>
 <wire x1="30.75" y1="65.75" x2="30.75" y2="63" width="0.15" layer="16"/>
-<wire x1="15.75" y1="48" x2="7.92" y2="48" width="0.15" layer="16"/>
-<wire x1="7.92" y1="48" x2="6.27" y2="46.35" width="0.15" layer="16"/>
 <wire x1="8.95" y1="49.03" x2="6.27" y2="46.35" width="0.15" layer="1"/>
 <wire x1="8.95" y1="49.03" x2="10.9762" y2="49.03" width="0.15" layer="1"/>
 <wire x1="11.0962" y1="46.59" x2="10.9762" y2="46.71" width="0.15" layer="1"/>
 <wire x1="10.9762" y1="46.71" x2="10.9762" y2="49.03" width="0.15" layer="1"/>
+<wire x1="14.1" y1="46.35" x2="6.27" y2="46.35" width="0.15" layer="16"/>
 </signal>
 <signal name="BOOT_0">

Commit message: eskd fixes
Parts:
- renumbered S1 to SB1
Changed lines of the file:
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@@
 <layer number="23" name="tOrigins" color="15" fill="1" visible="yes" active="yes"/>
 <layer number="24" name="bOrigins" color="15" fill="1" visible="yes" active="yes"/>
-<layer number="25" name="tNames" color="7" fill="1" visible="no" active="yes"/>
-<layer number="26" name="bNames" color="15" fill="1" visible="no" active="yes"/>
+<layer number="25" name="tNames" color="7" fill="1" visible="yes" active="yes"/>
+<layer number="26" name="bNames" color="15" fill="1" visible="yes" active="yes"/>
 <layer number="27" name="tValues" color="7" fill="1" visible="no" active="yes"/>
 <layer number="28" name="bValues" color="7" fill="1" visible="no" active="yes"/>
-<layer number="29" name="tStop" color="7" fill="3" visible="no" active="yes"/>
-<layer number="30" name="bStop" color="7" fill="6" visible="no" active="yes"/>
+<layer number="29" name="tStop" color="7" fill="3" visible="yes" active="yes"/>
+<layer number="30" name="bStop" color="7" fill="6" visible="yes" active="yes"/>
 <layer number="31" name="tCream" color="7" fill="4" visible="no" active="yes"/>
 <layer number="32" name="bCream" color="7" fill="5" visible="no" active="yes"/>
@@
 <attribute name="VALUE" x="90.19" y="38.405" size="0.8128" layer="27" ratio="10" rot="R270"/>
 </element>
-<element name="S1" library="switch" package="B3S-10XX" value="RESET" x="5" y="16" smashed="yes" rot="R270">
+<element name="SB1" library="switch" package="B3S-10XX" value="RESET" x="5" y="16" smashed="yes" rot="R270">
 <attribute name="LABEL" value="RESET" x="8.685" y="19.8575" size="1.6764" layer="25" ratio="18" rot="R270"/>
 <attribute name="PARTNO" value="4-1437565-2" x="5" y="16" size="1.778" layer="27" rot="R270" display="off"/>
@@
 <contactref element="C51" pad="2"/>
 <contactref element="C55" pad="2"/>
-<contactref element="S1" pad="2"/>
-<contactref element="S1" pad="1"/>
+<contactref element="SB1" pad="2"/>
+<contactref element="SB1" pad="1"/>
 <contactref element="XP1" pad="4"/>
 <contactref element="XP1" pad="6"/>
@@
 <contactref element="R9" pad="1"/>
 <contactref element="C2" pad="1"/>
-<contactref element="S1" pad="3"/>
-<contactref element="S1" pad="4"/>
+<contactref element="SB1" pad="3"/>
+<contactref element="SB1" pad="4"/>
 <contactref element="XP1" pad="15"/>
 <wire x1="2.75" y1="11.45" x2="2.75" y2="20.55" width="0.15" layer="1"/>

Commit message: nop
Parts:
- C3: value 0.1uF -> 10uF/10V; device rcl:C0603 -> rcl:A/3216-18W
- C4: value 10uF/10V -> 22pF; device rcl:A/3216-18W -> rcl:C0603
- C59: value 0.01uF -> 0.1uF
- C6: value 22pF -> 0.1uF
- C60: value 0.1uF -> 10uF/50V; device rcl:C0603 -> rcl:C2220K
- C61: value 10uF/50V -> 0.1uF; device rcl:C2220K -> rcl:C0603
- C62: value 0.1uF -> 0.01uF
- R10: value 0Ohm -> 10kOhm; device rcl:R0805 -> rcl:R0603
- R8: value 10kOhm -> 0Ohm; device rcl:R0603 -> rcl:R0805
- moved C6 44.0 mm to (11.8, 49.0), turned to 0 degrees
- moved R8 42.9 mm to (37.5, 78.5), turned to 270 degrees
- moved R10 40.9 mm to (11.9, 46.6), turned to 0 degrees
- moved C59 37.5 mm to (188.8, 55.2), turned to 270 degrees
- moved C2 32.1 mm to (28.0, 76.7), turned to 135 degrees
- moved C61 23.2 mm to (185.5, 25.8), turned to 180 degrees
- moved C3 21.4 mm to (46.2, 65.5), turned to 180 degrees
- moved C62 11.8 mm to (194.4, 18.1)
- moved C4 10.9 mm to (46.4, 76.4), turned to 135 degrees
- moved C60 10.2 mm to (194.9, 47.0), turned to 0 degrees
- moved C5 3.39 mm to (44.1, 78.9), turned to 315 degrees
- moved R9 2.46 mm to (11.9, 44.1)
Connections:
- net +24V_CLEAR: now also C59.1, C60.2, C61.1; no longer C60.1, C61.2, C62.1
- net +3V3: now also C2.1, C3.+, R10.2; no longer C3.1, C4.+, R8.2
- net AGND: now also R8.2; no longer R10.2
- net GND: now also C3.-, C4.2, C60.1, C62.2, R8.1; no longer C3.2, C4.-, C60.2, C61.1, R10.1
- net JTDO: now also R9.1; no longer R8.1
- net N$14: now also C5.1; no longer C6.1
- net N$15: now also C4.1; no longer C5.1
- net N$28: now also C62.1; no longer C59.1
- net N$86: now also C61.2; no longer C62.2
- net RST: now also C6.1, R10.1; no longer C2.1, R9.1
Routing:
- net GND: vias 120 -> 121

Commit message: before resizing board
Parts:
- added Z2: NFE31PT, emi-filter:NFE31
- moved C11 7.00 mm to (10.5, 72.2)
- moved R22 7.00 mm to (10.2, 68.0)
- moved R29 7.00 mm to (12.5, 69.5)
- moved DD2 6.50 mm to (5.00, 70.2)
- moved R12 3.00 mm to (5.50, 63.0)
- moved R14 3.00 mm to (5.50, 59.0)
- moved VD2 3.00 mm to (7.50, 61.0)
- moved XP3 3.00 mm to (3.00, 58.5)
- moved R11 2.50 mm to (5.75, 81.2)
- moved R13 2.50 mm to (5.75, 77.5)
- moved VD1 2.50 mm to (7.75, 79.2)
- moved XP2 2.50 mm to (3.00, 77.5)
Routing:
- net I2C_SCL: track 10.7 -> 17.2 mm
- net I2C_SDA: track 10.6 -> 17.1 mm
- net SPEEDOMETER: track 90.9 -> 96.1 mm
- net +5V: track 404.5 -> 409.6 mm
- net BOOT_0: track 37.9 -> 36.6 mm
- net BOOT_1: track 24.8 -> 25.8 mm
- net +3V3: track 831.9 -> 831.4 mm

Commit message: moved to different board
Parts:
- removed Z2: NFE31PT, emi-filter:NFE31
- added JP7, JP8: STAND-OFF-M4, mount:STAND-OFF
- JP1, JP2, JP3, JP4, JP5, JP6: value STAND-OFFLONG -> STAND-OFF-M4; device mount:STAND-OFF-LONG -> mount:STAND-OFF
- moved JP4 207.2 mm to (3.50, 75.0), turned to 0 degrees
- moved JP2 160.9 mm to (115.0, 3.50), turned to 0 degrees
- moved JP6 143.8 mm to (115.0, 146.5)
- moved JP5 124.4 mm to (226.5, 75.0), turned to 0 degrees
- moved C99 14.5 mm to (130.0, 87.3)
- moved R237 14.5 mm to (130.0, 90.5)
- moved R326 14.5 mm to (130.7, 63.0)
- moved VD112 14.5 mm to (137.3, 126.3)
- moved VD113 14.5 mm to (134.8, 126.3)
- moved VD114 14.5 mm to (132.3, 126.3)
- moved VD115 14.5 mm to (129.8, 126.3)
- moved C128 14.5 mm to (130.7, 66.2)
- moved C139 14.5 mm to (117.7, 64.4)
- moved C59 14.5 mm to (199.3, 65.2)
- moved R1 14.5 mm to (22.4, 41.1)
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Other:
- board size 210 x 132 mm -> 230 x 150 mm

Commit message: begin of EMI filtering adding
Parts:
- added Z20, Z21, Z22, Z23, Z24, Z25, Z26, Z27, Z28, Z29, Z30, Z31, Z32, Z33, Z34, Z35, Z36, Z37: NFE31PT, emi-filter:NFE31
- XP10, XP8, XP9: device connector:MOLEX-90130-*16 -> connector:MOLEX-90130-16
- XP11: device connector:MOLEX-90130-*34 -> connector:MOLEX-90130-34
- XP12, XP5, XP6: device connector:TYCO-174049(2.54) -> connector:MOLEX-90130-08
- XP4, XP7: device connector:TYCO-174053(2.54) -> connector:MOLEX-90130-16
- moved R363 48.5 mm to (20.5, 17.5)
- moved R364 48.5 mm to (18.8, 12.5)
- moved R365 48.5 mm to (17.8, 18.2)
- moved R366 48.5 mm to (20.0, 21.4)
- moved R367 48.5 mm to (15.8, 21.6)
- moved R368 48.5 mm to (18.0, 21.6)
- moved VD212 48.5 mm to (15.2, 16.5)
- moved VT3 48.5 mm to (23.8, 17.5)
- moved VT4 48.5 mm to (18.8, 15.2)
- moved R17 30.0 mm to (42.5, 29.0)
- moved R25 30.0 mm to (41.5, 32.0)
- moved XS1 28.8 mm to (6.00, 7.50), turned to 0 degrees
- moved R21 24.0 mm to (48.5, 40.0)
- moved R28 24.0 mm to (47.5, 37.0)
- moved L4 22.8 mm to (11.6, 9.25), turned to 0 degrees
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Connections:
- new net N$315: C12.1, R38.2, R46.2, Z20.1
- net AN_FILTERED_0: now also Z20.3; no longer C12.1, R38.2, R46.2
Routing:
- net N$229: track 6.96 -> 53.8 mm
- net +5V: track 409.6 -> 378.9 mm, vias 17 -> 15
- net USART_FROM_MCU: track 34.9 -> 4.28 mm
- net N$237: track 8.04 -> 38.5 mm
- net USART_TO_MCU: track 39.2 -> 9.18 mm
- net N$236: track 12.4 -> 42.3 mm
- net D+: track 42.1 -> 70.2 mm
- net D-: track 42.7 -> 70.4 mm
- net SPEEDOMETER: track 96.1 -> 122.5 mm
- net N$234: track 63.3 -> 37.8 mm
- net N$242: track 3.22 -> 27.2 mm
- net CAN_TX: track 32.0 -> 8.04 mm
- net N$314: track 5.59 -> 29.6 mm
- net CAN_RX: track 31.7 -> 7.66 mm
- net AN_FILTERED_0: track 43.1 -> 24.3 mm
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
Commit message: nop1
Parts:
- removed R17, R21, R25, R28: 100Ohm, rcl:R0603
- added VD213, VD214: SMBJ24CA, diode:SMB-BIDIR
- added Z10, Z11, Z12, Z13, Z14, Z15, Z16, Z17, Z18, Z19, Z2, Z3, Z38, Z39, Z4, Z40, Z41, Z42, Z43, Z44, Z45, Z46, Z47, Z48, Z49, Z5, Z6, Z7, Z8, Z9: NFE31PT, emi-filter:NFE31
- moved Z32 143.9 mm to (25.5, 95.0), turned to 270 degrees
- moved Z35 143.4 mm to (15.0, 91.0)
- moved Z23 141.4 mm to (60.5, 95.0), turned to 270 degrees
- moved Z33 140.8 mm to (18.5, 95.0), turned to 270 degrees
- moved Z29 140.3 mm to (32.5, 95.0), turned to 270 degrees
- moved Z27 137.3 mm to (46.5, 95.0), turned to 270 degrees
- moved Z26 137.2 mm to (39.5, 95.0), turned to 270 degrees
- moved Z24 136.4 mm to (57.0, 95.0), turned to 270 degrees
- moved Z31 135.7 mm to (29.0, 95.0), turned to 270 degrees
- moved Z30 135.6 mm to (22.0, 95.0), turned to 270 degrees
- moved Z21 134.7 mm to (64.0, 95.0), turned to 270 degrees
- moved Z34 131.9 mm to (15.0, 87.5)
- moved Z28 131.7 mm to (36.0, 95.0), turned to 270 degrees
- moved Z25 130.7 mm to (50.0, 95.0), turned to 270 degrees
- moved Z22 126.6 mm to (53.5, 95.0), turned to 270 degrees
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Connections:
- new net N$316: C13.1, R39.2, R47.2, Z21.1
- new net N$317: C14.1, R40.2, R48.2, Z22.1
- new net N$318: C15.1, R41.2, R49.2, Z23.1
- new net N$319: C16.1, R42.2, R50.2, Z24.1
- new net N$320: C17.1, R43.2, R51.2, Z25.1
- new net N$321: C18.1, R44.2, R52.2, Z26.1
- new net N$322: C19.1, R45.2, R53.2, Z27.1
- new net N$323: C20.1, R62.2, R70.2, Z28.1
- new net N$324: C21.1, R63.2, R71.2, Z29.1
- new net N$325: C22.1, R64.2, R72.2, Z30.1
- new net N$326: C23.1, R65.2, R73.2, Z31.1
- new net N$327: C24.1, R66.2, R74.2, Z32.1
- new net N$328: C25.1, R67.2, R75.2, Z33.1
- new net N$329: C26.1, R68.2, R76.2, Z34.1
- new net N$330: C27.1, R69.2, R77.2, Z35.1
- new net N$331: C8.2, DD1.19, DD1.20, R8.2, Z2.3
- new net N$332: R12.1, Z6.1
- new net N$333: R11.1, Z5.1
- new net N$334: R1.1, XP1.3, Z3.3
- new net N$335: R2.1, XP1.5, Z4.3
- new net N$336: R6.1, XP1.7, Z8.3
- new net N$337: C6.1, R10.1, SB1.3, SB1.4, XP1.15, Z10.3
- new net N$338: R7.1, XP1.9, Z7.3
- new net N$339: R9.1, XP1.13, Z9.3
- new net N$340: DD1.48, Z12.3
- new net N$341: DD2.6, R29.2, Z11.1
- new net N$342: DA15.5, Z37.1
- new net N$343: R368.2, Z36.1
- new net N$344: R367.2, Z19.1
- new net N$345: DA15.4, Z17.1
- new net N$346: DA15.6, Z18.1
- new net N$347: R130.2, R132.2, VD50.C, Z38.1
- new net N$348: R131.2, R133.2, VD51.C, Z39.1
- new net N$349: R134.2, VD52.C, Z40.1
- new net N$350: DD1.97, Z41.1
- new net N$351: R19.2, Z42.3
- new net N$352: R26.2, Z44.3
- new net N$353: R20.2, Z43.3
- new net N$354: R27.2, Z45.3
- new net N$355: R15.2, Z46.3
- new net N$356: R16.2, Z49.3
- new net N$357: R23.2, Z47.3
- new net N$358: R24.2, Z48.3
- net AGND: now also Z2.1; no longer C8.2, DD1.19, DD1.20, R8.2
- net AN_FILTERED_1: now also Z21.3; no longer C13.1, R39.2, R47.2
- net AN_FILTERED_10: now also Z30.3; no longer C22.1, R64.2, R72.2
- net AN_FILTERED_11: now also Z31.3; no longer C23.1, R65.2, R73.2
- net AN_FILTERED_12: now also Z32.3; no longer C24.1, R66.2, R74.2
- net AN_FILTERED_13: now also Z33.3; no longer C25.1, R67.2, R75.2
- net AN_FILTERED_14: now also Z34.3; no longer C26.1, R68.2, R76.2
- net AN_FILTERED_15: now also Z35.3; no longer C27.1, R69.2, R77.2
- net AN_FILTERED_2: now also Z22.3; no longer C14.1, R40.2, R48.2
- net AN_FILTERED_3: now also Z23.3; no longer C15.1, R41.2, R49.2
- net AN_FILTERED_4: now also Z24.3; no longer C16.1, R42.2, R50.2
- net AN_FILTERED_5: now also Z25.3; no longer C17.1, R43.2, R51.2
- net AN_FILTERED_6: now also Z26.3; no longer C18.1, R44.2, R52.2
- net AN_FILTERED_7: now also Z27.3; no longer C19.1, R45.2, R53.2
- net AN_FILTERED_8: now also Z28.3; no longer C20.1, R62.2, R70.2
- net AN_FILTERED_9: now also Z29.3; no longer C21.1, R63.2, R71.2
- net BOOT_0: now also Z6.3; no longer R12.1
- net BOOT_1: now also Z5.3; no longer R11.1
- net CAN_RX: now also DD1.81, Z15.3; no longer DA16.4, R28.1
- net CAN_TX: now also DD1.82, Z16.3; no longer DA16.1, R21.1
- net D+: now also Z18.3; no longer DA15.6
- net D-: now also Z17.3; no longer DA15.4
- net FREQMETER: now also Z39.3; no longer R131.2, R133.2, VD51.C
- net FROM_RS232: now also VD214.A2, Z14.1; no longer DA17.8
- net GND: now also VD213.A1, VD214.A1, Z10.2, Z11.2, Z12.2, Z13.2, Z14.2, Z15.2, Z16.2, Z17.2, Z18.2, Z19.2, Z2.2, Z20.2, Z21.2, Z22.2, Z23.2, Z24.2, Z25.2, Z26.2, Z27.2, Z28.2, Z29.2, Z3.2, Z30.2, Z31.2, Z32.2, Z33.2, Z34.2, Z35.2, Z36.2, Z37.2, Z38.2, Z39.2, Z4.2, Z40.2, Z41.2, Z42.2, Z43.2, Z44.2, Z45.2, Z46.2, Z47.2, Z48.2, Z49.2, Z5.2, Z6.2, Z7.2, Z8.2, Z9.2
- net I2C_SCL: now also Z11.3; no longer DD2.6, R29.2
- net I2C_SDA: now also Z12.1; no longer DD1.48
- net JTCK: now also Z7.1; no longer R7.1, XP1.9
- net JTDI: now also Z4.1; no longer R2.1, XP1.5
- net JTDO: now also Z9.1; no longer R9.1, XP1.13
- net JTMS: now also Z8.1; no longer R6.1, XP1.7
- net JTRST: now also Z3.1; no longer R1.1, XP1.3
- net N$16: now also Z46.1; no longer R15.2
- net N$220: now also Z47.1; no longer R23.2
- net N$221: now also Z49.1; no longer R16.2
- net N$222: now also Z48.1; no longer R24.2
- net N$223: now also Z42.1; no longer R19.2
- net N$229: now also Z37.3; no longer DA15.5
- net N$236: now also DA17.8, Z14.3; no longer DD1.68, R17.2
- net N$237: now also DA17.7, Z13.3; no longer DD1.69, R25.2
- net N$242: now also DA16.1, Z16.1; no longer DD1.82, R21.2
- net N$272: now also Z41.3; no longer DD1.97
- net N$275: now also Z44.1; no longer R26.2
- net N$276: now also Z43.1; no longer R20.2
- net N$277: now also Z45.1; no longer R27.2
- net N$314: now also DA16.4, Z15.1; no longer DD1.81, R28.2
- net RST: now also Z10.1; no longer C6.1, R10.1, SB1.3, SB1.4, XP1.15
- net SPEEDOMETER: now also Z40.3; no longer R134.2, VD52.C
- net TACHOMETER: now also Z38.3; no longer R130.2, R132.2, VD50.C
- net TO_RS232: now also VD213.A2, Z13.1; no longer DA17.7
- net USART_FROM_MCU: now also DD1.68; no longer R17.1
- net USART_TO_MCU: now also DD1.69; no longer R25.1
- net USB_DISCOVERY: now also Z36.3; no longer R368.2
- net USB_PRESENT: now also Z19.3; no longer R367.2
Routing:
- net N$277: track 114.6 -> 17.6 mm
- net N$354: track 0.00 -> 95.6 mm
- net N$337: track 0.00 -> 89.7 mm, vias 0 -> 2
- net SPEEDOMETER: track 122.5 -> 33.3 mm, vias 4 -> 2
- net N$349: track 0.00 -> 86.3 mm, vias 0 -> 2
- net +3V3: track 817.7 -> 902.7 mm, vias 19 -> 20
- net TACHOMETER: track 86.5 -> 18.6 mm, vias 5 -> 1
- net N$221: track 102.8 -> 35.3 mm, vias 3 -> 2
- net N$223: track 81.1 -> 15.0 mm, vias 3 -> 0
- net N$356: track 0.00 -> 66.0 mm, vias 0 -> 3
- net N$275: track 81.1 -> 16.1 mm, vias 3 -> 1
- net N$222: track 100.0 -> 35.3 mm, vias 3 -> 1
- net N$347: track 0.00 -> 64.1 mm, vias 0 -> 2
- net N$352: track 0.00 -> 64.0 mm, vias 0 -> 2
- net N$358: track 0.00 -> 63.6 mm, vias 0 -> 2
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