File: hard/pcb_main/main.brd (EAGLE design)
At the start: 230 x 150 mm, 868 parts

Commit message: nop
Routing:
- net +3V3: track 811.1 -> 811.9 mm
Changed lines of the file:
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@@
 <layer number="23" name="tOrigins" color="15" fill="1" visible="yes" active="yes"/>
 <layer number="24" name="bOrigins" color="15" fill="1" visible="yes" active="yes"/>
-<layer number="25" name="tNames" color="7" fill="1" visible="no" active="yes"/>
-<layer number="26" name="bNames" color="15" fill="1" visible="no" active="yes"/>
+<layer number="25" name="tNames" color="7" fill="1" visible="yes" active="yes"/>
+<layer number="26" name="bNames" color="15" fill="1" visible="yes" active="yes"/>
 <layer number="27" name="tValues" color="7" fill="1" visible="no" active="yes"/>
 <layer number="28" name="bValues" color="7" fill="1" visible="no" active="yes"/>
-<layer number="29" name="tStop" color="7" fill="3" visible="no" active="yes"/>
-<layer number="30" name="bStop" color="15" fill="6" visible="no" active="yes"/>
+<layer number="29" name="tStop" color="7" fill="3" visible="yes" active="yes"/>
+<layer number="30" name="bStop" color="15" fill="6" visible="yes" active="yes"/>
 <layer number="31" name="tCream" color="7" fill="4" visible="no" active="yes"/>
 <layer number="32" name="bCream" color="7" fill="5" visible="no" active="yes"/>
@@
 <layer number="46" name="Milling" color="3" fill="1" visible="no" active="yes"/>
 <layer number="47" name="Measures" color="7" fill="1" visible="no" active="yes"/>
-<layer number="48" name="Document" color="7" fill="1" visible="yes" active="yes"/>
+<layer number="48" name="Document" color="7" fill="1" visible="no" active="yes"/>
 <layer number="49" name="Reference" color="7" fill="1" visible="no" active="yes"/>
 <layer number="50" name="dxf" color="7" fill="1" visible="no" active="no"/>
@@
 <layer number="106" name="bPlate" color="7" fill="1" visible="no" active="yes"/>
 <layer number="107" name="Crop" color="7" fill="1" visible="no" active="yes"/>
-<layer number="116" name="Patch_BOT" color="9" fill="4" visible="yes" active="yes"/>
+<layer number="116" name="Patch_BOT" color="9" fill="4" visible="no" active="yes"/>
 <layer number="121" name="_tsilk" color="7" fill="1" visible="no" active="yes"/>
 <layer number="122" name="_bsilk" color="7" fill="1" visible="no" active="yes"/>
@@
 <element name="VT1" library="transistor-fet" package="DPAK" value="IRFR430" x="198.69" y="14.31" smashed="yes" rot="R90">
 <attribute name="PARTNO" value="IRFR430APBF" x="198.69" y="14.31" size="1.778" layer="27" rot="R90" display="off"/>
-<attribute name="NAME" x="202.03" y="13.61" size="1.016" layer="25" ratio="18"/>
+<attribute name="NAME" x="203.03" y="13.61" size="1.016" layer="25" ratio="18"/>
 <attribute name="VALUE" x="199.96" y="11.77" size="0.8128" layer="27" ratio="10" rot="R90"/>
 </element>
@@
 <element name="VD61" library="diode" package="DPAK" value="600V/6A" x="192" y="22" smashed="yes" rot="R270">
 <attribute name="PARTNO" value="IDD06SG60C" x="192" y="22" size="1.778" layer="27" rot="R270" display="off"/>
-<attribute name="NAME" x="188.905" y="22.705" size="1.016" layer="25" ratio="18" rot="R180"/>
+<attribute name="NAME" x="192.905" y="26.705" size="1.016" layer="25" ratio="18" rot="R180"/>
 <attribute name="VALUE" x="190.73" y="24.54" size="0.8128" layer="27" ratio="10" rot="R270"/>
 </element>
@@
 <wire x1="180.4266" y1="53.075" x2="184.325" y2="53.075" width="0.15" layer="16"/>
 <wire x1="180.4266" y1="60.695" x2="180.4266" y2="60.745" width="0.15" layer="16"/>
-<wire x1="2.25" y1="59.75" x2="2.25" y2="66.75" width="0.15" layer="1"/>
+<wire x1="2.25" y1="59.75" x2="2.25" y2="65.75" width="0.15" layer="1"/>
 <wire x1="4.5" y1="97.5" x2="3.5" y2="98.5" width="0.15" layer="1"/>
 <wire x1="4.5" y1="94.5" x2="4.5" y2="97.5" width="0.15" layer="1"/>
 <wire x1="8.2625" y1="94" x2="5" y2="94" width="0.15" layer="1"/>
-<wire x1="2.25" y1="66.75" x2="8" y2="72.5" width="0.15" layer="1"/>
-<wire x1="8" y1="72.5" x2="8" y2="81.5" width="0.15" layer="1"/>
+<wire x1="2.25" y1="65.75" x2="9" y2="72.5" width="0.15" layer="1"/>
+<wire x1="9" y1="72.5" x2="9" y2="80.5" width="0.15" layer="1"/>
 <via x="82" y="70.5" extent="1-16" drill="0.5"/>
 <wire x1="8.75" y1="95.7062" x2="8.75" y2="94.4875" width="0.15" layer="1"/>
@@
 <wire x1="4.5475" y1="93.5475" x2="5" y2="94" width="0.15" layer="1"/>
 <wire x1="5" y1="94" x2="4.5" y2="94.5" width="0.15" layer="1"/>
-<wire x1="8" y1="81.5" x2="4.5" y2="85" width="0.15" layer="1"/>
+<wire x1="9" y1="80.5" x2="4.5" y2="85" width="0.15" layer="1"/>
 <wire x1="4.5" y1="85" x2="4.5" y2="86" width="0.15" layer="1"/>
 <wire x1="4.5475" y1="86" x2="4.5475" y2="88.25" width="0.15" layer="1"/>
@@
 </signal>
 </signals>
+<errors>
+</errors>
 </board>
 </drawing>

Commit message: n contr
Parts:
- R1, R100, R170, R171, R172, R173, R174, R175, R176, R177, R178, R179, R180, R181, R182, R183, R184, R185, R188, R2, R221, R222, R223, R224, R225, R226, R227, R228, R229, R230, R231, R232, R233, R234, R235, R236, R269, R270, R271, R272, R273, R274, R275, R276, R277, R278, R279, R280, R281, R282, R283, R284, R3, R317, R318, R319, R320, R321, R322, R323, R324, R325, R326, R327, R328, R329, R330, R331, R332, R333, R359, R361, R4, R42, R43, R44, R45, R46, R47, R48, R49, R5, R6, R66, R67, R68, R69, R7, R70, R71, R72, R73, R8, R87, R88, R89, R9, R90, R92, R93, R94, R95, R97, R98, R99: value 10kOhm -> 10kOhm/1%
- R11, R12, R126, R127, R130, R34, R35, R36, R37, R38, R39, R40, R41, R58, R59, R60, R61, R62, R63, R64, R65, R83, R84, R85: value 100kOhm -> 100kOhm/1%
- R116: value 1kOhm -> 1kOhm/20%
- R124, R125, R134, R15, R154, R155, R156, R157, R158, R159, R160, R161, R162, R163, R164, R165, R166, R167, R168, R169, R186, R187, R205, R206, R207, R208, R209, R210, R211, R212, R213, R214, R215, R216, R217, R218, R219, R220, R25, R253, R254, R255, R256, R257, R258, R259, R260, R261, R262, R263, R264, R265, R266, R267, R268, R301, R302, R303, R304, R305, R306, R307, R308, R309, R310, R311, R312, R313, R314, R315, R316, R342, R343, R344, R345, R346, R347, R348, R349, R350, R351, R352, R353, R354, R355, R356, R357, R363, R364: value 1kOhm -> 1kOhm/5%
- R128, R129, R360: value 36kOhm -> 36kOhm/5%
- R13, R136, R137, R14, R20: value 330Ohm -> 330Ohm/5%
- R131: value 15kOhm -> 15kOhm/5%
- R132: value 82kOhm -> 82kOhm/5%
- R133: value 470kOhm -> 470kOhm/5%
- R135: value 3.3kOhm -> 3.3kOhm/5%
- R138, R139, R140, R141, R142, R143, R144, R145, R146, R147, R148, R149, R150, R151, R152, R153, R189, R190, R191, R192, R193, R194, R195, R196, R197, R198, R199, R200, R201, R202, R203, R204, R237, R238, R239, R240, R241, R242, R243, R244, R245, R246, R247, R248, R249, R250, R251, R252, R285, R286, R287, R288, R289, R290, R291, R292, R293, R294, R295, R296, R297, R298, R299, R300: value 4.7kOhm -> 4.7kOhm/5%
- R16, R17, R18, R19, R21, R22, R23, R24, R334, R335, R336, R337, R338, R339, R340, R341: value 100Ohm -> 100Ohm/5%
- R26, R27, R28, R29, R30, R31, R32, R33, R50, R51, R52, R53, R54, R55, R56, R57: value 1kOhm -> 1kOhm/1%
- R358: value 120Ohm -> 120Ohm/5%
- R362: value 47kOhm -> 47kOhm/5%
