File: hard/e4/e4.sch (EAGLE design)
At the start: 16 parts

Commit message: nop
Parts:
- XP1: value 2РМДТ33Б32Г5В1В -> 2РМДТ33Б32Ш5В1В
- XP2: value 2РМДТ27Б19Г5В1В -> 2РМТ22Б10Ш1В1В; device connector:GENERIC_19_XP -> connector:GENERIC_10_XP
- XP3: value 2РМДТ18Б4Ш5В1В -> 2РМДТ27Б19Ш5В1В; device connector:GENERIC_04_XP -> connector:GENERIC_19_XP
- XP4: value 2РМТ22Б10Г1В1В -> 2РМДТ18Б4Ш5В1В; device connector:GENERIC_10_XP -> connector:GENERIC_04_XP
- XS1: value 2РМДТ33Б32Ш5В1В -> 2РМДТ33Б32Г5В1В
- XS11: value 90142-0008 -> 2РМДТ27Б19Г5В1В; device connector:GENERIC_08_XS -> connector:GENERIC_19_XS; PARTNO 90142-0008 -> (none)
- XS12: value 2РМДТ27Б19Ш5В1В -> 2РМТ22Б10Г1В1В; device connector:GENERIC_19_XS -> connector:GENERIC_10_XS
- XS2: value 2РМТ22Б10Ш1В1В -> 90142-0016; device connector:GENERIC_10_XS -> connector:GENERIC_16_XS; PARTNO (none) -> 90142-0016
- XS6: value 90142-0016 -> 90142-0008; device connector:GENERIC_16_XS -> connector:GENERIC_08_XS; PARTNO 90142-0016 -> 90142-0008
- XS7: value 90142-0008 -> 90142-0016; device connector:GENERIC_08_XS -> connector:GENERIC_16_XS; PARTNO 90142-0008 -> 90142-0016
- XS8: value 90142-0016 -> 90142-0034; device connector:GENERIC_16_XS -> connector:GENERIC_34_XS; PARTNO 90142-0016 -> 90142-0034
- XS9: value 90142-0034 -> 90142-0008; device connector:GENERIC_34_XS -> connector:GENERIC_08_XS; PARTNO 90142-0034 -> 90142-0008
Connections:
- net +24V: now also XP4.1, XP4.2, XS9.2, XS9.4, XS9.6, XS9.8; no longer XP3.1, XP3.2, XS10.2, XS10.4, XS10.6, XS10.8
- net AN1: now also XS11.1, XS7.1; no longer XP2.1, XS8.1
- net AN10: now also XS11.10, XS7.10; no longer XP2.10, XS8.10
- net AN11: now also XS11.11, XS7.11; no longer XP2.11, XS8.11
- net AN12: now also XS11.12, XS7.12; no longer XP2.12, XS8.12
- net AN13: now also XS11.13, XS7.13; no longer XP2.13, XS8.13
- net AN14: now also XS11.14, XS7.14; no longer XP2.14, XS8.14
- net AN15: now also XS11.15, XS7.15; no longer XP2.15, XS8.15
- net AN16: now also XS11.16, XS7.16; no longer XP2.16, XS8.16
- net AN2: now also XS11.2, XS7.2; no longer XP2.2, XS8.2
- net AN3: now also XS11.3, XS7.3; no longer XP2.3, XS8.3
- net AN4: now also XS11.4, XS7.4; no longer XP2.4, XS8.4
- net AN5: now also XS11.5, XS7.5; no longer XP2.5, XS8.5
- net AN6: now also XS11.6, XS7.6; no longer XP2.6, XS8.6
- net AN7: now also XS11.7, XS7.7; no longer XP2.7, XS8.7
- net AN8: now also XS11.8, XS7.8; no longer XP2.8, XS8.8
- net AN9: now also XS11.9, XS7.9; no longer XP2.9, XS8.9
- net CAN_H: now also XP2.2, XS6.2; no longer XS2.2, XS7.2
- net CAN_L: now also XP2.1, XS6.1; no longer XS2.1, XS7.1
- net FREQUENCY1: now also XS10.3, XS12.3; no longer XP4.3, XS11.3
- net GND: now also XP4.3, XP4.4, XS9.1, XS9.3, XS9.5, XS9.7; no longer XP3.3, XP3.4, XS10.1, XS10.3, XS10.5, XS10.7
- net OUT_DRV1: now also XP3.1, XS8.1, XS8.4; no longer XS12.1, XS9.1, XS9.4
- net OUT_DRV2: now also XP3.3, XS8.5, XS8.8; no longer XS12.3, XS9.5, XS9.8
- net OUT_DRV3: now also XP3.5, XS8.12, XS8.9; no longer XS12.5, XS9.12, XS9.9
- net OUT_DRV4: now also XP3.7, XS8.13, XS8.16; no longer XS12.7, XS9.13, XS9.16
- net OUT_DRV5: now also XP3.9, XS8.17, XS8.20; no longer XS12.9, XS9.17, XS9.20
- net OUT_DRV6: now also XP3.11, XS8.21, XS8.24; no longer XS12.11, XS9.21, XS9.24
- net OUT_DRV7: now also XP3.13, XS8.25, XS8.28; no longer XS12.13, XS9.25, XS9.28
- net OUT_DRV8: now also XP3.15, XS8.29, XS8.32; no longer XS12.15, XS9.29, XS9.32
- net PHASE_1: now also XS10.2, XS12.2; no longer XP4.2, XS11.2
- net PHASE_2: now also XS10.4, XS12.4; no longer XP4.4, XS11.4
- net PHASE_3: now also XS10.6, XS12.6; no longer XP4.6, XS11.6
- net REL1: now also XP1.1, XS2.1; no longer XS1.1, XS3.1
- net REL10: now also XP1.10, XS2.10; no longer XS1.10, XS3.10
- net REL11: now also XP1.11, XS2.11; no longer XS1.11, XS3.11
- net REL12: now also XP1.12, XS2.12; no longer XS1.12, XS3.12
- net REL13: now also XP1.13, XS2.13; no longer XS1.13, XS3.13
- net REL14: now also XP1.14, XS2.14; no longer XS1.14, XS3.14
- net REL15: now also XP1.15, XS2.15; no longer XS1.15, XS3.15
- net REL16: now also XP1.16, XS2.16; no longer XS1.16, XS3.16
- net REL17: now also XP1.17, XS3.1; no longer XS1.17, XS4.1
- net REL18: now also XP1.18, XS3.2; no longer XS1.18, XS4.2
- net REL19: now also XP1.19, XS3.3; no longer XS1.19, XS4.3
- net REL2: now also XP1.2, XS2.2; no longer XS1.2, XS3.2
- net REL20: now also XP1.20, XS3.4; no longer XS1.20, XS4.4
- net REL21: now also XP1.21, XS3.5; no longer XS1.21, XS4.5
- net REL22: now also XP1.22, XS3.6; no longer XS1.22, XS4.6
- net REL23: now also XP1.23, XS3.7; no longer XS1.23, XS4.7
- net REL24: now also XP1.24, XS3.8; no longer XS1.24, XS4.8
- net REL25: now also XP1.25, XS3.9; no longer XS1.25, XS4.9
- net REL26: now also XP1.26, XS3.10; no longer XS1.26, XS4.10
- net REL27: now also XP1.27, XS3.11; no longer XS1.27, XS4.11
- net REL28: now also XP1.28, XS3.12; no longer XS1.28, XS4.12
- net REL29: now also XP1.29, XS3.13; no longer XS1.29, XS4.13
- net REL3: now also XP1.3, XS2.3; no longer XS1.3, XS3.3
- net REL30: now also XP1.30, XS3.14; no longer XS1.30, XS4.14
- net REL31: now also XP1.31, XS3.15; no longer XS1.31, XS4.15
- net REL32: now also XP1.32, XS3.16; no longer XS1.32, XS4.16
- net REL33: now also XS1.1, XS4.1; no longer XP1.1, XS5.1
- net REL34: now also XS1.2, XS4.2; no longer XP1.2, XS5.2
- net REL35: now also XS1.3, XS4.3; no longer XP1.3, XS5.3
- net REL36: now also XS1.4, XS4.4; no longer XP1.4, XS5.4
- net REL37: now also XS1.5, XS4.5; no longer XP1.5, XS5.5
- net REL38: now also XS1.6, XS4.6; no longer XP1.6, XS5.6
- net REL39: now also XS1.7, XS4.7; no longer XP1.7, XS5.7
- net REL4: now also XP1.4, XS2.4; no longer XS1.4, XS3.4
- net REL40: now also XS1.8, XS4.8; no longer XP1.8, XS5.8
- net REL41: now also XS1.9, XS4.9; no longer XP1.9, XS5.9
- net REL42: now also XS1.10, XS4.10; no longer XP1.10, XS5.10
- net REL43: now also XS1.11, XS4.11; no longer XP1.11, XS5.11
- net REL44: now also XS1.12, XS4.12; no longer XP1.12, XS5.12
- net REL45: now also XS1.13, XS4.13; no longer XP1.13, XS5.13
- net REL46: now also XS1.14, XS4.14; no longer XP1.14, XS5.14
- net REL47: now also XS1.15, XS4.15; no longer XP1.15, XS5.15
- net REL48: now also XS1.16, XS4.16; no longer XP1.16, XS5.16
- net REL49: now also XS1.17, XS5.1; no longer XP1.17, XS6.1
- net REL5: now also XP1.5, XS2.5; no longer XS1.5, XS3.5
- net REL50: now also XS1.18, XS5.2; no longer XP1.18, XS6.2
- net REL51: now also XS1.19, XS5.3; no longer XP1.19, XS6.3
- net REL52: now also XS1.20, XS5.4; no longer XP1.20, XS6.4
- net REL53: now also XS1.21, XS5.5; no longer XP1.21, XS6.5
- net REL54: now also XS1.22, XS5.6; no longer XP1.22, XS6.6
- net REL55: now also XS1.23, XS5.7; no longer XP1.23, XS6.7
- net REL56: now also XS1.24, XS5.8; no longer XP1.24, XS6.8
- net REL57: now also XS1.25, XS5.9; no longer XP1.25, XS6.9
- net REL58: now also XS1.26, XS5.10; no longer XP1.26, XS6.10
- net REL59: now also XS1.27, XS5.11; no longer XP1.27, XS6.11
- net REL6: now also XP1.6, XS2.6; no longer XS1.6, XS3.6
- net REL60: now also XS1.28, XS5.12; no longer XP1.28, XS6.12
- net REL61: now also XS1.29, XS5.13; no longer XP1.29, XS6.13
- net REL62: now also XS1.30, XS5.14; no longer XP1.30, XS6.14
- net REL63: now also XS1.31, XS5.15; no longer XP1.31, XS6.15
- net REL64: now also XS1.32, XS5.16; no longer XP1.32, XS6.16
- net REL7: now also XP1.7, XS2.7; no longer XS1.7, XS3.7
- net REL8: now also XP1.8, XS2.8; no longer XS1.8, XS3.8
- net REL9: now also XP1.9, XS2.9; no longer XS1.9, XS3.9
- net RS232_RX: now also XP2.3, XS6.3; no longer XS2.3, XS7.3
- net RS232_TX: now also XP2.4, XS6.4; no longer XS2.4, XS7.4
- net TACHOMETER: now also XS10.1, XS12.1; no longer XP4.1, XS11.1
- net VCC_DRV1: now also XP3.2, XS8.2, XS8.3; no longer XS12.2, XS9.2, XS9.3
- net VCC_DRV2: now also XP3.4, XS8.6, XS8.7; no longer XS12.4, XS9.6, XS9.7
- net VCC_DRV3: now also XP3.6, XS8.10, XS8.11; no longer XS12.6, XS9.10, XS9.11
- net VCC_DRV4: now also XP3.8, XS8.14, XS8.15; no longer XS12.8, XS9.14, XS9.15
- net VCC_DRV5: now also XP3.10, XS8.18, XS8.19; no longer XS12.10, XS9.18, XS9.19
- net VCC_DRV6: now also XP3.12, XS8.22, XS8.23; no longer XS12.12, XS9.22, XS9.23
- net VCC_DRV7: now also XP3.14, XS8.26, XS8.27; no longer XS12.14, XS9.26, XS9.27
- net VCC_DRV8: now also XP3.16, XS8.30, XS8.31; no longer XS12.16, XS9.30, XS9.31
Other:
- moved on the sheet: XP1, XS1, XS10, XS3, XS4, XS5

Commit message: nop
Other:
- note removed: "Crimp contacts 90119-2110 "Molex""
- note removed: "Make nets from MGTF-0.35 wire"
Changed lines of the file:
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@@
 <text x="186.69" y="319.405" size="1.524" layer="94" rot="MR0">AN_RAW_15</text>
 <text x="186.69" y="316.865" size="1.524" layer="94" rot="MR0">AN_RAW_16</text>
-<text x="17.78" y="15.24" size="3.048" layer="94" font="fixed">Make nets from MGTF-0.35 wire</text>
-<text x="17.78" y="10.16" size="3.048" layer="94" font="fixed">Crimp contacts 90119-2110 "Molex"</text>
 <text x="132.08" y="373.38" size="1.524" layer="94">KCAY.469555.025</text>
 <wire x1="104.14" y1="83.82" x2="104.14" y2="97.79" width="0.1524" layer="94"/>
@@
 <instance part="XS9" gate="G$1" x="198.12" y="175.26" smashed="yes" rot="MR0">
 <attribute name="NAME" x="193.04" y="180.34" size="1.524" layer="95"/>
-<attribute name="VALUE" x="205.74" y="153.67" size="1.524" layer="96" rot="MR0"/>
+<attribute name="VALUE" x="205.74" y="153.67" size="1.524" layer="96" font="fixed" rot="MR0"/>
 <attribute name="PARTNO" x="198.12" y="175.26" size="1.778" layer="96" rot="MR0" display="off"/>
 </instance>
 <instance part="XS2" gate="G$1" x="96.52" y="355.6" smashed="yes">
 <attribute name="NAME" x="101.6" y="360.68" size="1.524" layer="95" rot="MR0"/>
-<attribute name="VALUE" x="89.535" y="313.69" size="1.524" layer="96"/>
+<attribute name="VALUE" x="89.535" y="313.69" size="1.524" layer="96" font="fixed"/>
 <attribute name="PARTNO" x="96.52" y="355.6" size="1.778" layer="96" display="off"/>
 </instance>
 <instance part="XS3" gate="G$1" x="96.52" y="302.26" smashed="yes">
 <attribute name="NAME" x="101.6" y="307.34" size="1.524" layer="95" rot="MR0"/>
-<attribute name="VALUE" x="90.17" y="260.35" size="1.524" layer="96"/>
+<attribute name="VALUE" x="90.17" y="260.35" size="1.524" layer="96" font="fixed"/>
 <attribute name="PARTNO" x="96.52" y="302.26" size="1.778" layer="96" display="off"/>
 </instance>
 <instance part="XS4" gate="G$1" x="96.52" y="236.22" smashed="yes">
 <attribute name="NAME" x="101.6" y="241.3" size="1.524" layer="95" rot="MR0"/>
-<attribute name="VALUE" x="90.17" y="194.31" size="1.524" layer="96"/>
+<attribute name="VALUE" x="90.17" y="194.31" size="1.524" layer="96" font="fixed"/>
 <attribute name="PARTNO" x="96.52" y="236.22" size="1.778" layer="96" display="off"/>
 </instance>
 <instance part="XS5" gate="G$1" x="96.52" y="182.88" smashed="yes">
 <attribute name="NAME" x="101.6" y="187.96" size="1.524" layer="95" rot="MR0"/>
-<attribute name="VALUE" x="89.535" y="140.97" size="1.524" layer="96"/>
+<attribute name="VALUE" x="89.535" y="140.97" size="1.524" layer="96" font="fixed"/>
 <attribute name="PARTNO" x="96.52" y="182.88" size="1.778" layer="96" display="off"/>
 </instance>
 <instance part="XS7" gate="G$1" x="198.12" y="355.6" smashed="yes" rot="MR0">
 <attribute name="NAME" x="193.04" y="360.68" size="1.524" layer="95"/>
-<attribute name="VALUE" x="195.58" y="313.69" size="1.524" layer="96"/>
+<attribute name="VALUE" x="195.58" y="313.69" size="1.524" layer="96" font="fixed"/>
 <attribute name="PARTNO" x="198.12" y="355.6" size="1.778" layer="96" rot="MR0" display="off"/>
 </instance>
 <instance part="XS8" gate="G$1" x="198.12" y="284.48" smashed="yes" rot="MR0">
 <attribute name="NAME" x="193.04" y="289.56" size="1.524" layer="95"/>
-<attribute name="VALUE" x="195.58" y="196.85" size="1.524" layer="96"/>
+<attribute name="VALUE" x="195.58" y="196.85" size="1.524" layer="96" font="fixed"/>
 <attribute name="PARTNO" x="198.12" y="284.48" size="1.778" layer="96" rot="MR0" display="off"/>
 </instance>
 <instance part="XS10" gate="G$1" x="198.12" y="132.08" smashed="yes" rot="MR0">
 <attribute name="NAME" x="193.04" y="137.16" size="1.524" layer="95"/>
-<attribute name="VALUE" x="195.58" y="110.49" size="1.524" layer="96"/>
+<attribute name="VALUE" x="195.58" y="110.49" size="1.524" layer="96" font="fixed"/>
 <attribute name="PARTNO" x="198.12" y="132.08" size="1.778" layer="96" rot="MR0" display="off"/>
 </instance>
 <instance part="XS6" gate="G$1" x="96.52" y="116.84" smashed="yes">
 <attribute name="NAME" x="101.6" y="121.92" size="1.524" layer="95" rot="MR0"/>
-<attribute name="VALUE" x="88.9" y="95.25" size="1.524" layer="96"/>
+<attribute name="VALUE" x="88.9" y="95.25" size="1.524" layer="96" font="fixed"/>
 <attribute name="PARTNO" x="96.52" y="116.84" size="1.778" layer="96" display="off"/>
 </instance>
@@
 <instance part="XS1" gate="G$1" x="58.42" y="231.14" smashed="yes" rot="MR0">
 <attribute name="NAME" x="55.88" y="236.22" size="1.524" layer="95" rot="MR0"/>
-<attribute name="VALUE" x="53.34" y="148.59" size="1.524" layer="96" rot="MR0"/>
+<attribute name="VALUE" x="53.34" y="148.59" size="1.524" layer="96" font="fixed" rot="MR0"/>
 </instance>
 <instance part="XP1" gate="G$1" x="58.42" y="355.6" smashed="yes" rot="MR0">
 <attribute name="NAME" x="55.88" y="360.68" size="1.524" layer="95" rot="MR0"/>
-<attribute name="VALUE" x="53.34" y="273.05" size="1.524" layer="96" rot="MR0"/>
+<attribute name="VALUE" x="53.34" y="273.05" size="1.524" layer="96" font="fixed" rot="MR0"/>
 </instance>
 <instance part="XP2" gate="G$1" x="58.42" y="116.84" smashed="yes" rot="MR0">
 <attribute name="NAME" x="55.88" y="121.92" size="1.524" layer="95" rot="MR0"/>
-<attribute name="VALUE" x="53.34" y="90.17" size="1.524" layer="96" rot="MR0"/>
+<attribute name="VALUE" x="53.34" y="90.17" size="1.524" layer="96" font="fixed" rot="MR0"/>
 </instance>
 <instance part="XS11" gate="G$1" x="246.38" y="355.6" smashed="yes">
 <attribute name="NAME" x="248.92" y="360.68" size="1.524" layer="95"/>
-<attribute name="VALUE" x="251.46" y="306.07" size="1.524" layer="96"/>
+<attribute name="VALUE" x="251.46" y="306.07" size="1.524" layer="96" font="fixed"/>
 </instance>
 <instance part="XP3" gate="G$1" x="246.38" y="284.48" smashed="yes">
 <attribute name="NAME" x="248.92" y="289.56" size="1.524" layer="95"/>
-<attribute name="VALUE" x="251.46" y="234.95" size="1.524" layer="96"/>
+<attribute name="VALUE" x="251.46" y="234.95" size="1.524" layer="96" font="fixed"/>
 </instance>
 <instance part="XS12" gate="G$1" x="248.92" y="132.08" smashed="yes">
 <attribute name="NAME" x="251.46" y="137.16" size="1.524" layer="95"/>
-<attribute name="VALUE" x="254" y="105.41" size="1.524" layer="96"/>
+<attribute name="VALUE" x="254" y="105.41" size="1.524" layer="96" font="fixed"/>
 </instance>
 </instances>

Commit message: n contr fixes
Other:
- note added: "<< >>"
- note added: "<<+24V>>"
- note added: "<<AN>>"
- note added: "<<FRQ>>"
- note added: "<<OUT>>"
- note added: "<<REL1>>"
- note added: "<<REL2>>"
- note added: "<<RS232>>"
- note added: "XP1"
- note added: "XS1"
- note added: "XS2"
- note added: "XS3"
