File: hard/e4/e4.sch (EAGLE design)
At the start: 16 parts

Commit message: n contr
Parts:
- XP1: value 2РМДТ33Б32Ш5В1В -> (none)
- XP2: value 2РМТ22Б10Ш1В1В -> (none)
- XP3: value 2РМДТ27Б19Ш5В1В -> (none)
- XP4: value 2РМДТ18Б4Ш5В1В -> (none)
- XS1: value 2РМДТ33Б32Г5В1В -> (none)
- XS10, XS6, XS9: PARTNO 90142-0008 -> (none)
- XS11: value 2РМДТ27Б19Г5В1В -> (none)
- XS12: value 2РМТ22Б10Г1В1В -> (none)
- XS2, XS3, XS4, XS5, XS7: PARTNO 90142-0016 -> (none)
- XS8: PARTNO 90142-0034 -> (none)
Other:
- note removed: "1"
- note removed: "2"
- note removed: "3"
- note removed: "4"
- note removed: "5"
- note removed: "6"
- note removed: "7"
- note removed: "XP1"
- note removed: "XS1"
- note removed: "XS2"
- note removed: "XS3"
