File: hard/mpiovd/mpiovd.sch (EAGLE design)
At the start: 868 parts

Commit message: n contr
Connections:
- net AGND: now also Z5.3; no longer Z5.1
- net BOOT_0: now also Z10.1; no longer Z10.3
- net BOOT_1: now also Z9.1; no longer Z9.3
- net I2C_SCL: now also Z11.1; no longer Z11.3
- net I2C_SDA: now also Z17.3; no longer Z17.1
- net JTCK: now also Z7.3; no longer Z7.1
- net JTDI: now also Z6.3; no longer Z6.1
- net JTDO: now also Z4.3; no longer Z4.1
- net JTMS: now also Z3.3; no longer Z3.1
- net JTRST: now also Z2.3; no longer Z2.1
- net N$331: now also Z5.1; no longer Z5.3
- net N$332: now also Z10.3; no longer Z10.1
- net N$333: now also Z9.3; no longer Z9.1
- net N$334: now also Z2.1; no longer Z2.3
- net N$335: now also Z6.1; no longer Z6.3
- net N$336: now also Z3.1; no longer Z3.3
- net N$337: now also Z8.1; no longer Z8.3
- net N$338: now also Z7.1; no longer Z7.3
- net N$339: now also Z4.1; no longer Z4.3
- net N$340: now also Z17.1; no longer Z17.3
- net N$341: now also Z11.3; no longer Z11.1
- net RST: now also Z8.3; no longer Z8.1
Other:
- moved on the sheet: C69, C70, C71, C72, C73, C74, C75, C76, C77, C78, C79, C80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

Commit message: fixed XP12 connector description
Parts:
- XP12: PARTNO 90142-0008 -> 90130-1208
